Commit message: Update arm.xacro

File: arm_description/urdf/arm.xacro (robot description, xacro)
@@ -7,6 +7,6 @@
    <inertial>
     <origin xyz="-0.002716977299773592 1.9808719046125134e-13 -0.002500000000000375" rpy="0 0 0"/>
-    <mass value="2"/>
-    <inertia ixx="7.2e-05" iyy="7.6e-05" izz="0.000147" ixy="-0.0" iyz="0.0" ixz="-0.04"/>
+    <mass value="150"/>
+    <inertia ixx="10" iyy="10" izz="15" ixy="0" iyz="0.0" ixz="-10"/>
   </inertial>
   <visual>
@@ -27,6 +27,6 @@
   <inertial>
     <origin xyz="-0.1170701569437167 0.05258495071306836 0.24677061589144064" rpy="0 0 0"/>
-    <mass value="0.6560949347888712"/>
-    <inertia ixx="0.020432" iyy="0.024363" izz="0.005288" ixy="0.000756" iyz="-0.001594" ixz="0.009271"/>
+    <mass value="1.5"/>
+    <inertia ixx="0.20432" iyy="0.24363" izz="0.5288" ixy="0.456" iyz="-0.1594" ixz="0.9271"/>
   </inertial>
   <visual>
@@ -47,6 +47,6 @@
   <inertial>
     <origin xyz="0.0912652794492105 -0.04755997480137449 0.15715086928559246" rpy="0 0 0"/>
-    <mass value="0.4295491979731537"/>
-    <inertia ixx="0.0092" iyy="0.01219" izz="0.003285" ixy="0.00233" iyz="0.000401" ixz="-0.005183"/>
+    <mass value="1"/>
+    <inertia ixx="0.52" iyy="0.1219" izz="0.3285" ixy="0.233" iyz="0.401" ixz="-0.5183"/>
   </inertial>
   <visual>
@@ -67,6 +67,6 @@
   <inertial>
     <origin xyz="0.012554620120246197 2.599084142351771e-13 0.021619020423368274" rpy="0 0 0"/>
-    <mass value="0.03924999999999999"/>
-    <inertia ixx="7e-06" iyy="9e-06" izz="3e-06" ixy="0.0" iyz="0.0" ixz="-3e-06"/>
+    <mass value="0.3"/>
+    <inertia ixx="0.05" iyy="0.05" izz="0.03" ixy="0.0" iyz="0.0" ixz="0.1"/>
   </inertial>
   <visual>
@@ -87,6 +87,6 @@
   <inertial>
     <origin xyz="-0.00379841512801708 -4.326319553927361e-16 0.05885490789415437" rpy="0 0 0"/>
-    <mass value="0.2699874429831712"/>
-    <inertia ixx="0.000593" iyy="0.000639" izz="0.0003" ixy="0.0" iyz="-0.0" ixz="-1.7e-05"/>
+    <mass value="1"/>
+    <inertia ixx="0.5" iyy="0.639" izz="0.3" ixy="0.0" iyz="-0.0" ixz="0.01"/>
   </inertial>
   <visual>
